File: Phase_B/ArduinoShieldThermoPro/ArduinoShieldThermoPro.kicad_pcb (KiCad board)
At the start: 2 copper layers, 68.6 x 53.3 mm, 23 parts, among them J1 Power, J2 Digital/PWM, J3 Analog, J4 Digital/PWM, J5 CONN_GYRO, J6 CONN_DISPLSAY, SW1 SW_SPST, SW2 SW_SPST, SW3 SW_SPST, SW4 SW_SPST, SW5 SW_SPST

Commit message: Update PCB
Parts:
- removed MH1, MH2, MH3, MH4: MountingHole_3.2mm, Arduino_MountingHole:MountingHole_3.2mm
- added J7: CONN_TEMP, Connector_JST:JST_XH_B3B-XH-A_1x03_P2.50mm_Vertical, F.Cu at (139.5, 55.6)
- R1, R2, R3, R4, R5, R6: footprint Resistor_THT:R_Axial_DIN0411_L9.9mm_D3.6mm_P15.24mm_Horizontal -> Resistor_THT:R_Axial_DIN0207_L6.3mm_D2.5mm_P10.16mm_Horizontal
- moved J6 48.1 mm to (111.7, 69.1), turned to 90 degrees
- moved SW3 44.5 mm to (157.3, 71.1), turned to 90 degrees
- moved SW2 44.3 mm to (157.3, 61.3), turned to 90 degrees
- moved R6 43.9 mm to (133.0, 52.3), turned to -90 degrees
- moved R1 40.3 mm to (141.8, 92.9), turned to 180 degrees
- moved R2 29.1 mm to (141.6, 85.0), turned to 180 degrees
- moved J5 28.6 mm to (104.3, 64.0)
- moved R3 28.4 mm to (141.9, 89.1), turned to 180 degrees
- moved SW4 26.3 mm to (136.7, 61.5)
- moved SW5 22.7 mm to (134.3, 73.5)
- moved R4 20.0 mm to (143.5, 69.6), turned to 180 degrees
- moved SW1 19.4 mm to (157.2, 81.3), turned to 90 degrees
- moved D1 18.5 mm to (128.8, 55.2), turned to 180 degrees
- moved R5 18.4 mm to (141.7, 81.6), turned to 180 degrees
- moved RV1 3.35 mm to (152.1, 90.3), turned to -90 degrees
Connections:
- J2 pad 10: /8 -> /Temp_Digital
- J4 pad 5: /Button_lock -> /Button_light
- R3 pad 1: /Button_cal -> /Button_light
- SW3 pad 1: /Button_cal -> /Button_light
Routing:
- net +5V: track 0.00 -> 170.2 mm
- net /Button_onoff: track 0.00 -> 53.6 mm
- net /Button_light: track 0.00 -> 51.3 mm
- net /Button_units: track 0.00 -> 48.7 mm
- net /Button_cal: track 0.00 -> 45.0 mm
- net /Button_lock: track 0.00 -> 31.0 mm
- net /I2C_SCL: track 0.00 -> 28.3 mm
- net /I2C_SDA: track 0.00 -> 28.3 mm
- net Net-(D1-A): track 0.00 -> 10.6 mm
- net /LED_Light: track 0.00 -> 7.44 mm
- net /Temp_Digital: track 0.00 -> 6.54 mm
- net /Temp_Sensor: track 0.00 -> 6.18 mm
- added copper zone on B.Cu, net GND
Other:
- board text removed: "ICSP"
