File: Phase_B/ArduinoShieldThermoPro/ArduinoShieldThermoPro.kicad_sch (KiCad schematic)
At the start: 19 parts, among them J1 Power, J2 Digital/PWM, J3 Analog, J4 Digital/PWM, J5 CONN_GYRO, J6 CONN_DISPLSAY, SW1 SW_SPST, SW2 SW_SPST, SW3 SW_SPST, SW4 SW_SPST, SW5 SW_SPST

Commit message: Update PCB
Parts:
- added J7: CONN_TEMP, Connector_JST:JST_XH_B3B-XH-A_1x03_P2.50mm_Vertical, symbol Connector_Generic:Conn_01x03
- R1, R2, R3, R4, R5, R6: footprint Resistor_THT:R_Axial_DIN0411_L9.9mm_D3.6mm_P15.24mm_Horizontal -> Resistor_THT:R_Axial_DIN0207_L6.3mm_D2.5mm_P10.16mm_Horizontal
Connections:
- net +5V: now also J7.3 (Pin_3)
- net Button_cal: no longer R3.1, SW3.1 (A)
- net Button_lock: no longer J4.5 (Pin_5)
- net GND: now also J7.1 (Pin_1)
- net 8 renamed Temp_Digital
- net Temp_Digital: now also J7.2 (Pin_2)
- new net Button_light: J4.5 (Pin_5), R3.1, SW3.1 (A)
- no-connect marks 21 -> 20
Other:
- note added: "8"
- note added: "DS18B20 (Temp Sesnsor)"
